File: ATMEGA Power Circuit/ATMEGA Power Circuit.kicad_pcb (KiCad board)
At the start: 4 copper layers, 65 x 30 mm, 32 parts, among them J1 Conn_01x03, J2 ICSP, J3 Screw_Terminal_01x02, J4 Screw_Terminal_01x02, J5 Raspberry_Pi_2_3, Q1 BSS138, Q2 BSS138, U1 ATmega328P-A, U2 ds3231sn-, U3 TPS2557DRBR, U4 XC6206P332MR

Commit message: update KiCad files to Rev 0.1
Parts:
- added C10: 1.0 uf, Capacitor_SMD:C_0603_1608Metric_Pad1.08x0.95mm_HandSolder, F.Cu at (117.7, 47.8)
- added C9: 1.0 uf, Capacitor_SMD:C_0603_1608Metric_Pad1.08x0.95mm_HandSolder, F.Cu at (123.2, 47.8)
- added D2: B5819W SL, PCM_JLCPCB:D_SOD-123, F.Cu at (120.2, 50.7)
- added D3: Red, PCM_JLCPCB:D_0603, F.Cu at (123.6, 67.8)
- added R10: 10K, Resistor_SMD:R_0603_1608Metric_Pad0.98x0.95mm_HandSolder, F.Cu at (119.8, 67.8)
- added R11: 10K, Resistor_SMD:R_0603_1608Metric_Pad0.98x0.95mm_HandSolder, F.Cu at (78.2, 62.8)
- added R8: 100k, Resistor_SMD:R_0603_1608Metric_Pad0.98x0.95mm_HandSolder, F.Cu at (68.9, 51.6)
- added R9: 22k1, Resistor_SMD:R_0603_1608Metric_Pad0.98x0.95mm_HandSolder, F.Cu at (75.0, 51.4)
- BT1: value CR2032_Battery_Cell -> CR2032
- C6: moved to B.Cu
- C7: value 1.0 uf -> 100uF; footprint Capacitor_SMD:C_0603_1608Metric_Pad1.08x0.95mm_HandSolder -> PCM_JLCPCB:C_CASE-B-3528-21(mm)
- C8: value 1.0 uf -> 100n; footprint Capacitor_SMD:C_0603_1608Metric_Pad1.08x0.95mm_HandSolder -> Capacitor_SMD:C_0402_1005Metric_Pad0.74x0.62mm_HandSolder
- R4: value 10K -> 4k7; moved to B.Cu
- R5: value 10K -> 0; footprint Resistor_SMD:R_0603_1608Metric_Pad0.98x0.95mm_HandSolder -> Jumper:SolderJumper-2_P1.3mm_Open_Pad1.0x1.5mm; moved to B.Cu
- R6: value 100k -> 10K
- R7: value 22k1 -> 10K
- UART: renamed from J1; value Conn_01x03 -> Conn_01x04; footprint Connector_PinHeader_2.54mm:PinHeader_1x03_P2.54mm_Vertical -> Connector_PinHeader_2.54mm:PinHeader_1x04_P2.54mm_Vertical
- moved C7 48.1 mm to (73.4, 48.1), turned to 0 degrees
- moved C8 43.5 mm to (71.3, 54.3), turned to 180 degrees
- moved C6 27.0 mm to (96.1, 63.1), turned to 0 degrees
- moved R4 26.3 mm to (100.2, 62.8), turned to -90 degrees
- moved R5 24.0 mm to (100.7, 58.8)
- moved R6 10.1 mm to (79.0, 48.2), turned to 0 degrees
- moved R2 5.63 mm to (106.4, 51.1)
- moved Q1 5.03 mm to (106.2, 48.4)
- moved R7 4.80 mm to (79.0, 46.6), turned to 0 degrees
- moved U4 2.97 mm to (120.4, 47.8)
- moved Q2 2.28 mm to (109.8, 48.4)
- moved UART 2.12 mm to (114.1, 67.0)
- moved U3 1.96 mm to (71.8, 51.7)
- moved R1 1.57 mm to (109.9, 51.1)
- moved C1 0.82 mm to (121.0, 54.2), turned to 0 degrees
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- renumbered J2 to ICSP
Connections:
- C6 pad 1: /LOAD_SW_IN -> +3V3
- C7 pad 1: GND -> /LOAD_SW_OUT
- C7 pad 2: Vin -> GND
- C8 pad 1: +3V3 -> /LOAD_SW_IN
- R4 pad 1: +3V3_PI -> +3V3
- R4 pad 2: /SDA_PI -> /SQW
- R5 pad 1: +3V3_PI -> Net-(U2-*RST)
- R5 pad 2: /SCL_PI -> GND
- R6 pad 1: /LOAD_SW_IN -> +3V3_PI
- R6 pad 2: Net-(U3-~{FAULT}) -> /SDA_PI
- R7 pad 1: Net-(U3-ILIM) -> +3V3_PI
- R7 pad 2: GND -> /SCL_PI
- U2 pad 4: unconnected-(U2-*RST-Pad4) -> Net-(U2-*RST)
Routing:
- net GND: track 50.3 -> 64.8 mm, vias 28 -> 33
- net +3V3: track 71.1 -> 82.2 mm
- net /SCL_PI: track 38.4 -> 28.9 mm, vias 2 -> 0
- net Net-(U2-*RST): track 0.00 -> 8.53 mm
- net /LOAD_SW_IN: track 13.2 -> 7.28 mm
- net /LOAD_SW_EN: track 57.8 -> 60.5 mm
- net +3V3_PI: track 27.6 -> 25.3 mm
- net /SDA_PI: track 32.6 -> 34.8 mm, vias 2 -> 0
- net Net-(D3-Pad2): track 0.00 -> 2.10 mm
- net /UART_TX: track 6.83 -> 8.29 mm
- net /UART_RX: track 7.76 -> 9.02 mm
- net /SDA_SLV: track 27.6 -> 28.6 mm
- net Vin: track 9.60 -> 10.2 mm
- net /SQW: track 22.3 -> 22.9 mm
- net /SCL_SLV: track 29.0 -> 29.6 mm
Other:
- board text added: "Evan L 2025/07/02 Rev. 0.1 SEJJ Programmable RTC Pwr Switch"
- board text added: "GND"
- board text added: "ICSP"
- board text added: "PI PWR"
- board text added: "RX"
- board text added: "TX"
- board text added: "U2 RST"
- board text added: "UART"
- board text added: "VIN"
- board text removed: "SEJJ Programmable RTC Pwr Switch"
